File: FemtoFC.kicad_sch (KiCad schematic)
At the start: 29 parts, among them J3 Micro_SD_Card, P1 USB_C_Plug_USB2.0, U1 USBLC6-2SC6, U3 ATSAMD21G18A-M, U4 W25Q128JVS, Y1 Crystal

Commit message: 0.2
PCB edit
Added 3D models
Changed lines of the file:
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@@
     (pin "2")
   )
-  (sheet (at 251.46 17.78) (size 27.94 8.89) (fields_autoplaced)
+  (sheet (at 251.46 19.05) (size 27.94 7.62) (fields_autoplaced)
     (stroke (width 0.1524) (type solid) (color 0 0 0 0))
     (fill (color 0 0 0 0.0000))
-    (property "Sheet name" "Pyro" (id 0) (at 251.46 17.0684 0)
+    (property "Sheet name" "Pyro" (id 0) (at 251.46 18.3384 0)
       (effects (font (size 1.27 1.27)) (justify left bottom))
     )
@@
     )
   )
-  (sheet (at 252.73 52.07) (size 26.67 6.35) (fields_autoplaced)
+  (sheet (at 251.46 50.8) (size 27.94 7.62) (fields_autoplaced)
     (stroke (width 0.1524) (type solid) (color 0 0 0 0))
     (fill (color 0 0 0 0.0000))
-    (property "Sheet name" "PSU" (id 0) (at 252.73 51.3584 0)
+    (property "Sheet name" "PSU" (id 0) (at 251.46 50.0884 0)
       (effects (font (size 1.27 1.27)) (justify left bottom))
     )
-    (property "Sheet file" "psu.kicad_sch" (id 1) (at 252.73 59.0046 0)
+    (property "Sheet file" "psu.kicad_sch" (id 1) (at 251.46 59.0046 0)
       (effects (font (size 1.27 1.27)) (justify left top))
     )
@@
       (reference "#PWR0156") (unit 1) (value "GND") (footprint "")
     )
+    (path "/0332463b-8e2a-4e73-a08f-934bcf12edb1/ce581da9-ac1a-4c11-bedb-fb991b651d4d"
+      (reference "#PWR0157") (unit 1) (value "GND") (footprint "")
+    )
+    (path "/0332463b-8e2a-4e73-a08f-934bcf12edb1/1a9b102b-f5b0-4dd5-8cd5-3e35908dc054"
+      (reference "#PWR0158") (unit 1) (value "+BATT") (footprint "")
+    )
+    (path "/0332463b-8e2a-4e73-a08f-934bcf12edb1/446d393f-e711-4111-885c-286518d34313"
+      (reference "BZ1") (unit 1) (value "Buzzer") (footprint "Buzzer_Beeper:Buzzer_Murata_PKMCS0909E")
+    )
     (path "/84f4a80d-ac01-4c0e-a15b-9186acd006b1/266746d7-7ad0-435d-bc4d-678b9195d0ee"
       (reference "C1") (unit 1) (value "100nF") (footprint "Capacitor_SMD:C_0603_1608Metric_Pad1.08x0.95mm_HandSolder")
@@
       (reference "Q2") (unit 2) (value "FDS4953") (footprint "Package_SO:SOIC-8_3.9x4.9mm_P1.27mm")
     )
+    (path "/0332463b-8e2a-4e73-a08f-934bcf12edb1/24d7c602-2a97-48b3-9837-d97ee32b4712"
+      (reference "Q3") (unit 1) (value "NDT3055L") (footprint "Package_TO_SOT_SMD:TSOT-23_HandSoldering")
+    )
     (path "/84f4a80d-ac01-4c0e-a15b-9186acd006b1/a73fdb88-5cf1-4d10-95af-bbefd3332968"
       (reference "R1") (unit 1) (value "22k") (footprint "Resistor_SMD:R_0603_1608Metric_Pad0.98x0.95mm_HandSolder")
@@
       (reference "R16") (unit 1) (value "10k") (footprint "Resistor_SMD:R_0603_1608Metric_Pad0.98x0.95mm_HandSolder")
     )
+    (path "/0332463b-8e2a-4e73-a08f-934bcf12edb1/b6758490-44ba-4031-8cc3-20cb7d77e27d"
+      (reference "R17") (unit 1) (value "10k") (footprint "Resistor_SMD:R_0603_1608Metric_Pad0.98x0.95mm_HandSolder")
+    )
     (path "/e36f1f60-bcd7-4dd1-81ba-22b0a7500da2"

Commit message: Rework for prototype 2
Connections:
- net GND: now also C2.1, U3.18 (GND), U3.35 (GND), U3.42 (GND), U3.49 (EP)
- net VMeas: now reaches U3.11 (PA06)
Other:
- moved on the sheet: C2
Changed lines of the file:
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@@
 (kicad_sch (version 20211123) (generator eeschema)
   (paper "A4")
+  (junction (at 104.14 193.04) (diameter 0) (color 0 0 0 0)
+  )
   (junction (at 200.66 134.62) (diameter 0) (color 0 0 0 0)
   )
@@
     (stroke (width 0) (type default) (color 0 0 0 0))
   )
-  (wire (pts (xy 104.14 182.88) (xy 104.14 195.58))
-    (stroke (width 0) (type default) (color 0 0 0 0))
-  )
   (wire (pts (xy 200.66 132.08) (xy 200.66 134.62))
     (stroke (width 0) (type default) (color 0 0 0 0))
@@
     (stroke (width 0) (type default) (color 0 0 0 0))
   )
-  (wire (pts (xy 90.17 195.58) (xy 104.14 195.58))
+  (wire (pts (xy 90.17 193.04) (xy 104.14 193.04))
     (stroke (width 0) (type default) (color 0 0 0 0))
   )
@@
     (stroke (width 0) (type default) (color 0 0 0 0))
   )
+  (wire (pts (xy 90.17 185.42) (xy 90.17 186.69))
+    (stroke (width 0) (type default) (color 0 0 0 0))
+  )
   (wire (pts (xy 92.71 29.21) (xy 102.87 29.21))
     (stroke (width 0) (type default) (color 0 0 0 0))
@@
   )
   (wire (pts (xy 209.55 127) (xy 200.66 127))
+    (stroke (width 0) (type default) (color 0 0 0 0))
+  )
+  (wire (pts (xy 104.14 182.88) (xy 104.14 193.04))
     (stroke (width 0) (type default) (color 0 0 0 0))
   )
@@
     )
   )
+  (global_label "VMeas" (shape input) (at 86.36 109.22 180) (fields_autoplaced)
+    (effects (font (size 1.27 1.27)) (justify right))
+    (property "Intersheet References" "${INTERSHEET_REFS}" (id 0) (at 78.1412 109.1406 0)
+      (effects (font (size 1.27 1.27)) (justify right) hide)
+    )
+  )
   (global_label "MISO" (shape input) (at 86.36 142.24 180) (fields_autoplaced)
     (effects (font (size 1.27 1.27)) (justify right))
@@
     (pin "1")
   )
-  (symbol (lib_id "Device:C") (at 90.17 191.77 180) (unit 1)
-    (in_bom yes) (on_board yes)
-    (property "Reference" "C2" (id 0) (at 86.36 191.77 0)
-      (effects (font (size 1.27 1.27)) (justify left))
-    )
-    (property "Value" "10uF" (id 1) (at 86.36 189.23 0)
-      (effects (font (size 1.27 1.27)) (justify left))
-    )
-    (property "Footprint" "Capacitor_SMD:C_0603_1608Metric_Pad1.08x0.95mm_HandSolder" (id 2) (at 89.2048 187.96 0)
-      (effects (font (size 1.27 1.27)) hide)
-    )
-    (property "Datasheet" "~" (id 3) (at 90.17 191.77 0)
+  (symbol (lib_id "Device:C") (at 90.17 189.23 180) (unit 1)
+    (in_bom yes) (on_board yes)
+    (property "Reference" "C2" (id 0) (at 86.36 189.23 0)
+      (effects (font (size 1.27 1.27)) (justify left))
+    )
+    (property "Value" "10uF" (id 1) (at 86.36 186.69 0)
+      (effects (font (size 1.27 1.27)) (justify left))
+    )
+    (property "Footprint" "Capacitor_SMD:C_0603_1608Metric_Pad1.08x0.95mm_HandSolder" (id 2) (at 89.2048 185.42 0)
+      (effects (font (size 1.27 1.27)) hide)
+    )
+    (property "Datasheet" "~" (id 3) (at 90.17 189.23 0)
       (effects (font (size 1.27 1.27)) hide)
     )
@@
     (pin "1")
     (pin "2")
+  )
+  (symbol (lib_id "power:GND") (at 101.6 182.88 0) (unit 1)
+    (in_bom yes) (on_board yes)
+    (property "Reference" "#PWR0159" (id 0) (at 101.6 189.23 0)
+      (effects (font (size 1.27 1.27)) hide)
+    )
+    (property "Value" "GND" (id 1) (at 99.7459 186.7323 0)
+      (effects (font (size 1.27 1.27)) (justify left))
+    )
+    (property "Footprint" "" (id 2) (at 101.6 182.88 0)
+      (effects (font (size 1.27 1.27)) hide)
+    )
+    (property "Datasheet" "" (id 3) (at 101.6 182.88 0)
+      (effects (font (size 1.27 1.27)) hide)
+    )
+    (pin "1")
   )
   (symbol (lib_id "power:GND") (at 231.14 139.7 270) (unit 1)
@@
     (pin "1")
   )
-  (symbol (lib_id "power:+3.3V") (at 90.17 187.96 0) (unit 1)
-    (in_bom yes) (on_board yes)
-    (property "Reference" "#PWR0116" (id 0) (at 90.17 191.77 0)
-      (effects (font (size 1.27 1.27)) hide)
-    )
-    (property "Value" "+3.3V" (id 1) (at 87.63 182.88 0)
-      (effects (font (size 1.27 1.27)) (justify left))
-    )
-    (property "Footprint" "" (id 2) (at 90.17 187.96 0)
-      (effects (font (size 1.27 1.27)) hide)
-    )
-    (property "Datasheet" "" (id 3) (at 90.17 187.96 0)
+  (symbol (lib_id "power:+3.3V") (at 90.17 186.69 0) (unit 1)
+    (in_bom yes) (on_board yes)
+    (property "Reference" "#PWR0116" (id 0) (at 90.17 190.5 0)
+      (effects (font (size 1.27 1.27)) hide)
+    )
+    (property "Value" "+3.3V" (id 1) (at 87.63 181.61 0)
+      (effects (font (size 1.27 1.27)) (justify left))
+    )
+    (property "Footprint" "" (id 2) (at 90.17 186.69 0)
+      (effects (font (size 1.27 1.27)) hide)
+    )
+    (property "Datasheet" "" (id 3) (at 90.17 186.69 0)
       (effects (font (size 1.27 1.27)) hide)
     )
@@
     (pin "9")
   )
+  (symbol (lib_id "power:GND") (at 104.14 193.04 0) (unit 1)
+    (in_bom yes) (on_board yes)
+    (property "Reference" "#PWR0160" (id 0) (at 104.14 199.39 0)
+      (effects (font (size 1.27 1.27)) hide)
+    )
+    (property "Value" "GND" (id 1) (at 102.2859 196.8923 0)
+      (effects (font (size 1.27 1.27)) (justify left))
+    )
+    (property "Footprint" "" (id 2) (at 104.14 193.04 0)
+      (effects (font (size 1.27 1.27)) hide)
+    )
+    (property "Datasheet" "" (id 3) (at 104.14 193.04 0)
+      (effects (font (size 1.27 1.27)) hide)
+    )
+    (pin "1")
+  )
   (symbol (lib_id "Memory_Flash:W25Q128JVS") (at 260.35 91.44 0) (unit 1)
     (in_bom yes) (on_board yes) (fields_autoplaced)
@@
       (reference "#PWR0158") (unit 1) (value "+BATT") (footprint "")
     )
+    (path "/4dde0652-c37e-4ee1-a713-8f8df8324a53"
+      (reference "#PWR0159") (unit 1) (value "GND") (footprint "")
+    )
+    (path "/a9a62418-f170-4964-850f-1e89a1d2d04a"
+      (reference "#PWR0160") (unit 1) (value "GND") (footprint "")
+    )
     (path "/0332463b-8e2a-4e73-a08f-934bcf12edb1/446d393f-e711-4111-885c-286518d34313"
       (reference "BZ1") (unit 1) (value "Buzzer") (footprint "Buzzer_Beeper:Buzzer_Murata_PKMCS0909E")
@@
       (reference "R17") (unit 1) (value "10k") (footprint "Resistor_SMD:R_0603_1608Metric_Pad0.98x0.95mm_HandSolder")
     )
+    (path "/0332463b-8e2a-4e73-a08f-934bcf12edb1/4a06368c-ac2a-4bd5-acce-393b80f8a278"
+      (reference "R18") (unit 1) (value "1k") (footprint "Resistor_SMD:R_0603_1608Metric_Pad0.98x0.95mm_HandSolder")
+    )
     (path "/e36f1f60-bcd7-4dd1-81ba-22b0a7500da2"

Commit message: V3
Parts:
- removed FB1: FerriteBead_Small, Resistor_SMD:R_0805_2012Metric, symbol Device:FerriteBead_Small
- C10, C11, C12, C5, C6, C7, C8: footprint Capacitor_SMD:C_0603_1608Metric_Pad1.08x0.95mm_HandSolder -> Capacitor_SMD:C_0402_1005Metric_Pad0.74x0.62mm_HandSolder
- C2: value 10uF -> 1uF; footprint Capacitor_SMD:C_0603_1608Metric_Pad1.08x0.95mm_HandSolder -> Capacitor_SMD:C_0402_1005Metric_Pad0.74x0.62mm_HandSolder
- C4: value 100nF -> 1uF; footprint Capacitor_SMD:C_0603_1608Metric_Pad1.08x0.95mm_HandSolder -> Capacitor_SMD:C_0402_1005Metric_Pad0.74x0.62mm_HandSolder
- C9: value 100nF -> 10uF; footprint Capacitor_SMD:C_0603_1608Metric_Pad1.08x0.95mm_HandSolder -> Capacitor_SMD:C_0402_1005Metric_Pad0.74x0.62mm_HandSolder
- R3, R4, R5, R6, R7, R8, R9: footprint Resistor_SMD:R_0603_1608Metric_Pad0.98x0.95mm_HandSolder -> Resistor_SMD:R_0402_1005Metric_Pad0.72x0.64mm_HandSolder
Connections:
- net VDDANA is gone; now on net +3V3: C5.1, C6.1, U3.6 (VDDANA)
- net +3V3: no longer C2.2
- net GND: now also C2.2; no longer C2.1, P1.S1 (SHIELD)
- net MISO: now also U3.21 (PA12); no longer U3.28 (PA19), U4.2 (DO(IO1))
- net MOSI: now also U3.19 (PB10); no longer U3.25 (PA16), U4.5 (DI(IO0))
- net P1_EN: now also U3.27 (PA18); no longer U3.20 (PB11)
- net P2_EN: now also U3.28 (PA19); no longer U3.19 (PB10)
- net SCK: now also U3.20 (PB11); no longer U3.26 (PA17), U4.6 (CLK)
- net SCL: now also U3.32 (PA23); no longer U3.8 (PB09)
- net SDA: now also U3.31 (PA22); no longer U3.7 (PB08)
- net SPI_CS_FLASH: now also U3.39 (PA27); no longer U3.22 (PA13)
- net A4: now reaches U3.10 (PA05)
- net Buzzer: now reaches U3.13 (PA08)
- net D3: now reaches U3.14 (PA09)
- net A0: now reaches U3.3 (PA02)
- net FLASH_MOSI: now reaches U3.37 (PB22)
- net FLASH_MOSI: now also U4.5 (DI(IO0))
- net FLASH_SCK: now reaches U3.38 (PB23)
- net FLASH_SCK: now also U4.6 (CLK)
- net AREF: now reaches U3.4 (PA03)
- net AREF: now also C2.1
- net FLASH_MISO: now reaches U3.48 (PB03)
- net FLASH_MISO: now also U4.2 (DO(IO1))
- net A3: now reaches U3.9 (PA04)
- no-connect marks 2 -> 15
Other:
- moved on the sheet: R9, U3, U4

Commit message: Rev 27052023
Parts:
- removed C11, C12: 22pF, Capacitor_SMD:C_0402_1005Metric_Pad0.74x0.62mm_HandSolder, symbol Device:C
- removed Y1: Crystal, Crystal:Crystal_SMD_3215-2Pin_3.2x1.5mm, symbol Device:Crystal
- added R19, R20: 10k, Resistor_SMD:R_0402_1005Metric_Pad0.72x0.64mm_HandSolder, symbol Device:R
Connections:
- net +3V3: now also R19.1, R20.1
- net SCL: now also R20.2
- net SDA: now also R19.2
- net CI: now reaches U3.1 (PA00)
- net DI: now reaches U3.2 (PA01)
Other:
- note added: "Flash"
- note added: "MCU"
- note added: "MCU Decoupling"
- note added: "SD card"
- moved on the sheet: C10, C9, J3, R3, R4, R5, R6, R7, R8, U3
